Commit message: Modified laser_frame to laser

File: description/lidar.xacro (robot description, xacro)
@@ -3,8 +3,8 @@
     <joint name="laser_joint" type="fixed">
         <parent link="chassis"/>
-        <child link="laser_frame"/>
+        <child link="laser"/>
         <origin xyz="0.1 0 0.175" rpy="0 0 0"/>
     </joint>
-    <link name="laser_frame">
+    <link name="laser">
         <visual>
             <geometry>
@@ -22,5 +22,5 @@
         </xacro:inertial_cylinder>
     </link>
-    <gazebo reference="laser_frame">
+    <gazebo reference="laser">
         <material>Gazebo/Red</material>
         <sensor name="laser" type="ray">
@@ -46,5 +46,5 @@
                 </ros>
                 <output_type>sensor_msgs/LaserScan</output_type>
-                <frame_name>laser_frame</frame_name>
+                <frame_name>laser</frame_name>
             </plugin>
         </sensor>

Commit message: All changes fixed

File: description/lidar.xacro (robot description, xacro)
@@ -3,15 +3,8 @@
     <joint name="laser_joint" type="fixed">
         <parent link="chassis"/>
-<<<<<<< HEAD
         <child link="laser"/>
         <origin xyz="0.1 0 0.175" rpy="0 0 0"/>
     </joint>
     <link name="laser">
-=======
-        <child link="laser_frame"/>
-        <origin xyz="0.1 0 0.175" rpy="0 0 0"/>
-    </joint>
-    <link name="laser_frame">
->>>>>>> 4850b517a346bb38a1e334b50f5ddc5cb98ba943
         <visual>
             <geometry>
@@ -29,9 +22,5 @@
         </xacro:inertial_cylinder>
     </link>
-<<<<<<< HEAD
     <gazebo reference="laser">
-=======
-    <gazebo reference="laser_frame">
->>>>>>> 4850b517a346bb38a1e334b50f5ddc5cb98ba943
         <material>Gazebo/Red</material>
         <sensor name="laser" type="ray">
@@ -57,9 +46,5 @@
                 </ros>
                 <output_type>sensor_msgs/LaserScan</output_type>
-<<<<<<< HEAD
                 <frame_name>laser</frame_name>
-=======
-                <frame_name>laser_frame</frame_name>
->>>>>>> 4850b517a346bb38a1e334b50f5ddc5cb98ba943
             </plugin>
         </sensor>

File: description/robot.urdf.xacro (robot description, xacro)
@@ -2,8 +2,5 @@
 <robot xmlns:xacro="http://www.ros.org/wiki/xacro"  name="robot">
     <xacro:include filename="robot_core.xacro" />
-<<<<<<< HEAD
     <xacro:include filename="inertial_macros.xacro" />
-=======
->>>>>>> 4850b517a346bb38a1e334b50f5ddc5cb98ba943
     <xacro:include filename="gazebo_control.xacro" />
     <xacro:include filename="lidar.xacro" />
